File: rgb-secamfm500.brd (EAGLE design)
At the start: 89.5 x 47.6 mm, 104 parts

Commit message: .
Parts:
- added C10, C15, C18: 2n2, rcl:C0805K
- added C11, C13, C8: 56, rcl:C0805K
- added C14, C6, C7: 100, rcl:C0805K
- added C16: 50m, rcl:E2,5-6
- added C17: 33, rcl:C0805K
- added C2: 360, rcl:C0805K
- added L2A, L2B: (no value), Разъёмы штырьковые 2.54мм:1X01
- added R27, R28, R31: 330, rcl:M0805
- added R29, R30: 620, rcl:M0805
- added R33: 1k5, rcl:M0805
- added R34: 1k, rcl:M0805
- added R35: 3k3, rcl:M0805
- added VD1, VD3, VD4, VD5: КД521, diode:D-7.5
- added VT2: КТ315, m_transistor:TO92
- C12: value (none) -> 8..30
- moved R21 209.5 mm to (73.0, 119.4), flipped to the bottom, turned to 90 degrees
- moved R22 200.7 mm to (66.7, 119.4), flipped to the bottom, turned to 90 degrees
- moved R23 188.1 mm to (60.3, 113.0), flipped to the bottom, turned to 90 degrees
- moved R15 182.9 mm to (54.0, 119.4), flipped to the bottom, turned to 90 degrees
- moved DD4 58.4 mm to (92.1, 46.4)
Connections:
- new net N$100: L2A.1, VT2.2
- new net N$101: DD1.8, R33.2
- new net N$102: R35.2, VD4.C, VD6.C
- new net N$91: C6.2, C7.1, R21.2
- new net N$92: C13.2, DD4.14, L1.P$2, R27.2
- new net N$93: C12.1, L1.P$1
- new net N$94: C17.2, VD5.C, VT2.3
- new net N$95: C14.1, DD4.15, R28.2, R29.2
- new net N$96: C14.2, R30.2, R31.2, VT2.1
- new net N$97: R29.1, R30.1
- new net N$98: R28.1, R31.1
- net A: now also C10.1, C11.1, C13.1, C16.+, C17.1, C18.2, C8.1, DD4.1, DD4.16, L2B.1, VD5.A
- net GND: now also C16.-, C18.1, C7.2, DD4.8, R34.1, R35.1; no longer DD4.1, DD4.16
- net N$54: now also C6.1, DD1.9, R33.1, R34.2, VD4.A
- net N$80: now also C8.2, DD4.4, DD4.6, R15.2, VD1.C
- net N$85: now also C10.2, DD4.12, DD4.5
- net N$86: now also C11.2, C12.2, DD4.13, R27.1; no longer DD4.4, DD4.6, R15.2
- net N$88: now also C2.2
- net N$89: now also C2.1, VD1.A, VD3.A
- net VCC: no longer DD4.8
Routing:
- net N$85: track 0.00 -> 7.62 mm
- net A: track 0.00 -> 7.62 mm

Commit message: .
Parts:
- removed DD1', DD1'''': 74LS04N, 74xx-eu:DIL14
- removed R10', R10'', R10''', R10'''', R10'1: 15k, rcl:M0805
- removed R11', R11'', R11''', R11'''', R11'1: 7k5, rcl:M0805
- removed R12', R12'', R12''', R12'''', R12'1, R4', R4'', R4''', R4'''', R4'1, R7', R7'', R7''', R7'''', R7'1: 5k1, rcl:M0805
- removed R13', R13'''', R13'1, R13'2, R13'3: 3k3, rcl:M0805
- removed R5', R5'', R5''', R5'''', R5'1: 10k, rcl:M0805
- removed R6', R6'', R6''', R6'''', R6'1: 27k, rcl:M0805
- removed R8', R8'', R8''', R8'''', R8'1: 33k, rcl:M0805
- removed R9', R9'', R9''', R9'''', R9'1: 6k2, rcl:M0805
- added R32: 620, rcl:M0805
- moved L2A 11.6 mm to (112.4, 58.4), turned to 0 degrees
- moved L2B 2.54 mm to (110.5, 53.3), turned to 0 degrees
- moved R27 1.42 mm to (90.2, 60.3)
- moved C11 0.90 mm to (92.1, 57.8)
- moved C13 0.63 mm to (88.3, 57.8)
Connections:
- removed net N$1: R4''''.2, R5''''.2, R6''''.2
- removed net N$10: R10'.1, R5'.1, R7'.1
- removed net N$101: DD1.8, R33.2
- removed net N$11: DD1''''.2, R10''''.1, R5''''.1, R7''''.1
- removed net N$12: R7''''.2, R8''''.2, R9''''.2
- removed net N$13: DD1''''.4, R11''''.1, R4''''.1
- removed net N$14: DD1''''.3, R9''''.1
- removed net N$15: R10''''.2, R11''''.2, R12''''.2, R13''''.2
- removed net N$16: DD1''''.6, R6''''.1
- removed net N$17: DD1''''.5, R12''''.1, R8''''.1
- removed net N$18: R4'1.2, R5'1.2, R6'1.2
- removed net N$19: R12'1.1
- removed net N$2: R4'.2, R5'.2, R6'.2
- removed net N$20: R4''.2, R5''.2, R6''.2
- removed net N$21: R7'1.2, R8'1.2, R9'1.2
- removed net N$22: R9'1.1
- removed net N$23: R8'1.1
- removed net N$24: R10'1.2, R11'1.2, R12'1.2, R13'1.2
- removed net N$25: R5'1.1
- removed net N$26: R10'1.1
- removed net N$27: R7'1.1
- removed net N$28: R4'1.1
- removed net N$29: R6'1.1
- removed net N$3: DD1'.1, R11'.1, R4'.1
- removed net N$30: R11'1.1
- removed net N$31: R7''.2, R8''.2, R9''.2
- removed net N$32: R9''.1
- removed net N$33: R8''.1
- removed net N$34: R10''.2, R11''.2, R12''.2, R13'2.2
- removed net N$35: R5''.1
- removed net N$36: R10''.1
- removed net N$37: R7''.1
- removed net N$38: R4''.1
- removed net N$39: R6''.1
- removed net N$4: R7'.2, R8'.2, R9'.2
- removed net N$40: R11''.1
- removed net N$41: R12''.1
- removed net N$42: R4'''.2, R5'''.2, R6'''.2
- removed net N$43: R7'''.2, R8'''.2, R9'''.2
- removed net N$44: R7'''.1
- removed net N$45: R9'''.1
- removed net N$46: R10'''.2, R11'''.2, R12'''.2, R13'3.2
- removed net N$47: R4'''.1
- removed net N$48: R10'''.1
- removed net N$49: R8'''.1
- removed net N$5: DD1'.5, R6'.1
- removed net N$50: R5'''.1
- removed net N$51: R6'''.1
- removed net N$52: R11'''.1
- removed net N$53: R12'''.1
- removed net N$6: R10'.2, R11'.2, R12'.2, R13'.2
- removed net N$7: DD1'.2, R9'.1
- removed net N$8: DD1'.6, R12'.1, R8'.1
- removed net N$9: DD1''''.1
- removed net VCC: DD1''''.14, DD1'.14
- net GND: no longer DD1''''.7, DD1'.7, R13''''.1, R13'.1, R13'1.1, R13'2.1, R13'3.1
- net N$102: now also C15.2
- net N$83: now also C15.1, R32.1, VD3.C
- net N$97: now also R32.2
- net N$98: now also DD1.8, R33.2
Routing:
- net N$92: track 0.00 -> 7.31 mm
- net N$86: track 0.00 -> 6.03 mm
- net A: track 7.62 -> 9.43 mm

Commit message: .
Parts:
- removed !SJ1, !SJ2, !SJ3, SJ1, SJ2, SJ3: (no value), jumper:SJ
- added !J1, !J2, !J3, J1, J2, J3: (no value), jumper:SJ
- added R36: 620, rcl:M0805
- C3, C4: device rcl:C0805K -> rcl:C0805
- R20: device rcl:M0805 -> rcl:0207/12
- moved C2 113.8 mm to (94.0, 34.9), turned to 0 degrees
- moved VD4 110.7 mm to (39.4, 46.4)
- moved C8 108.2 mm to (83.2, 39.4), turned to 0 degrees
- moved C15 97.1 mm to (58.1, 56.5), turned to 0 degrees
- moved C10 93.5 mm to (83.2, 41.9), turned to 0 degrees
- moved R34 91.4 mm to (62.5, 58.7), turned to 0 degrees
- moved C7 90.5 mm to (92.1, 29.8), turned to 0 degrees
- moved R21 88.9 mm to (91.4, 32.4), turned to 0 degrees
- moved C6 88.9 mm to (83.2, 30.5), turned to 0 degrees
- moved R15 88.0 mm to (92.1, 40.0), turned to 0 degrees
- moved R22 86.8 mm to (83.8, 34.3), turned to 0 degrees
- moved VD3 85.9 mm to (101.6, 38.1), turned to 270 degrees
- moved VD1 85.9 mm to (94.6, 38.1), turned to 0 degrees
- moved R35 85.6 mm to (55.6, 65.1), turned to 270 degrees
- moved R33 84.9 mm to (61.3, 61.3), turned to 0 degrees
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Connections:
- net GND: now also C9.1, R36.2; no longer C9.2
- net N$57: now also !J1.1; no longer !SJ1.1
- net N$58: now also !J1.2, J1.2; no longer !SJ1.2, SJ1.2
- net N$59: now also !J2.2, J2.2; no longer !SJ2.2, SJ2.2
- net N$60: now also !J2.1; no longer !SJ2.1
- net N$61: now also J3.1; no longer SJ3.1
- net N$62: now also !J3.1; no longer !SJ3.1
- net N$63: now also J1.1; no longer SJ1.1
- net N$66: now also J2.1; no longer SJ2.1
- net N$67: now also !J3.2, J3.2; no longer !SJ3.2, SJ3.2
- net N$72: now also C9.2; no longer C9.1
- net N$92: now also R36.1
Routing:
- net N$72: track 0.00 -> 27.3 mm
- net GND: track 34.4 -> 54.5 mm
- net A: track 9.43 -> 22.9 mm
- net N$77: track 0.00 -> 10.5 mm
- net N$81: track 0.00 -> 9.74 mm
- net N$71: track 0.00 -> 6.77 mm
- net N$73: track 0.00 -> 6.45 mm
- net N$82: track 0.00 -> 3.38 mm
- net N$69: track 2.57 -> 5.87 mm
- net N$70: track 0.00 -> 2.99 mm
- net N$75: track 0.00 -> 2.54 mm
- net N$58: track 0.00 -> 2.54 mm
- net N$67: track 0.00 -> 2.54 mm
- net N$59: track 0.00 -> 2.54 mm
- net N$66: track 0.00 -> 2.41 mm
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
Commit message: .
Parts:
- moved VD6 1.85 mm to (44.8, 44.8)
- moved VD4 1.80 mm to (38.1, 45.1)
- moved R26 0.32 mm to (42.9, 73.0), turned to 180 degrees
- renumbered R19 to R19*
Connections:
- removed net N$72: C9.2, DD2.13, R18.1, R26.1, VD2.A
- new net N$1: DD2.13, R18.1, R26.2
- net N$81: now also C9.2, R26.1, VD2.A; no longer R26.2
Routing:
- net N$78: track 0.00 -> 31.3 mm
- net N$1: track 0.00 -> 27.4 mm
- net N$72: track 27.3 -> 0.00 mm
- net A: track 22.9 -> 36.8 mm
- net N$64: track 10.8 -> 21.0 mm
- net N$65: track 10.8 -> 12.3 mm
- net GND: track 54.5 -> 55.2 mm

Commit message: .
Parts:
- DD4: value К500ЛП216 -> К500ЛП216R; device 500:DIL16 -> 500:DIL16B
- R15: device rcl:M0805 -> rcl:0207/12
- moved L2A 38.3 mm to (76.2, 70.8)
- moved L2B 34.4 mm to (80.3, 69.8)
- moved R36 17.7 mm to (82.5, 62.9), turned to 0 degrees
- moved R21 15.6 mm to (81.6, 44.5), turned to 270 degrees
- moved C7 15.1 mm to (82.5, 41.6), turned to 180 degrees
- moved VD3 13.7 mm to (103.2, 51.8)
- moved C10 13.7 mm to (93.0, 51.4), turned to 180 degrees
- moved R16 13.0 mm to (69.5, 44.1)
- moved C8 12.4 mm to (89.2, 50.2), turned to 180 degrees
- moved C6 10.7 mm to (79.7, 40.6), turned to 90 degrees
- moved C2 10.6 mm to (97.2, 45.1)
- moved R22 10.2 mm to (83.8, 44.5), turned to 270 degrees
- moved R23 8.80 mm to (87.0, 44.8)
- moved R15 7.44 mm to (96.8, 45.7), flipped to the top, turned to 180 degrees
- moved C13 6.87 mm to (84.5, 52.1), turned to 90 degrees
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Connections:
- new net N$2: R32.1, VD3.C
- net N$83: no longer R32.1, VD3.C
Routing:
- net N$2: track 0.00 -> 26.2 mm
- net N$89: track 0.00 -> 20.0 mm
- net N$88: track 0.00 -> 19.9 mm
- net N$80: track 0.00 -> 13.9 mm
- net N$85: track 7.62 -> 20.3 mm
- net GND: track 55.2 -> 67.0 mm
- net A: track 36.8 -> 47.8 mm
- net N$95: track 0.00 -> 7.32 mm
- net N$92: track 7.31 -> 14.6 mm
- net N$90: track 0.00 -> 5.27 mm
- net N$86: track 6.03 -> 10.4 mm
- net N$91: track 0.00 -> 1.93 mm

Commit message: .
Parts:
- added L2: (no value), rcl:0204/5
- moved R13 64.6 mm to (80.3, 16.2), turned to 0 degrees
- moved B 47.7 mm to (77.2, 9.21)
- moved R6 47.0 mm to (65.4, 18.1)
- moved R8 43.1 mm to (74.3, 18.1), turned to 270 degrees
- moved G 42.8 mm to (82.9, 10.2)
- moved R5 41.6 mm to (63.2, 18.1)
- moved R12 39.0 mm to (72.1, 18.1), turned to 270 degrees
- moved R10 35.4 mm to (61.0, 18.1)
- moved R11 34.2 mm to (69.8, 18.1)
- moved R7 33.4 mm to (58.7, 18.1)
- moved R9 32.3 mm to (76.5, 18.1), turned to 270 degrees
- moved R4 29.3 mm to (67.6, 18.1)
- moved R 13.7 mm to (47.9, 21.0)
- moved C9 10.6 mm to (48.9, 69.2)
- moved VT2 8.94 mm to (65.7, 71.8), turned to 0 degrees
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Routing:
- net N$55: track 0.00 -> 25.7 mm
- net N$56: track 0.00 -> 18.2 mm
- net N$58: track 2.54 -> 16.2 mm
- net N$62: track 2.41 -> 15.2 mm
- net N$59: track 2.54 -> 14.2 mm
- net N$54: track 0.00 -> 4.45 mm
- net GND: track 67.0 -> 70.5 mm
- net N$79: track 0.00 -> 3.31 mm
- net N$65: track 12.3 -> 15.6 mm
- net N$81: track 9.72 -> 12.7 mm
- net N$86: track 10.4 -> 8.66 mm
- net N$92: track 14.6 -> 13.0 mm
- net N$95: track 7.32 -> 6.03 mm
- net N$85: track 20.3 -> 19.5 mm
- net A: track 47.8 -> 47.3 mm

Commit message: ..
Parts:
- added C19: 50m, rcl:E2,5-6
- added C20: 100n, rcl:C0805K
- DD4: value К500ЛП216R -> К500ЛП216
- R37: value 8* -> 8(20r)*
- moved C16 46.5 mm to (60.0, 79.1)
- moved L2 15.0 mm to (69.5, 80.0)
- moved R37 0.71 mm to (20.6, 47.0), turned to 180 degrees
- moved C17 0.32 mm to (67.0, 65.7)
Connections:
- new net B: C10.1, C11.1, C13.1, C16.+, C17.1, C18.2, C8.1, DD4.1, DD4.16, L2.2, L2B.1, VD5.A
- net A: now also C19.+, C20.1, L2.1, R37.2; no longer C10.1, C11.1, C13.1, C16.+, C17.1, C18.2, C8.1, DD4.1, DD4.16, L2B.1, R37.1, VD5.A
- net GND: now also C19.-, C20.2, C9.2; no longer C9.1
- net N$102: now also VD4.A; no longer VD4.C
- net N$54: now also VD4.C; no longer VD4.A
- net N$76: now also R37.1; no longer R37.2
- net N$81: now also C9.1; no longer C9.2
Routing:
- net A: track 47.3 -> 24.2 mm
- net B: track 0.00 -> 12.4 mm
- net N$81: track 12.7 -> 14.6 mm
- net GND: track 70.5 -> 72.4 mm
