File: rgb-secamfm500.sch (EAGLE design)
At the start: 104 parts

Commit message: .
Parts:
- added C10, C15, C18: 2n2, rcl:C-EUC0805K
- added C11, C13, C8: 56, rcl:C-EUC0805K
- added C14, C6, C7: 100, rcl:C-EUC0805K
- added C16: 50m, rcl:CPOL-EUE2.5-6
- added C17: 33, rcl:C-EUC0805K
- added C2: 360, rcl:C-EUC0805K
- added L2A, L2B: (no value), Разъёмы штырьковые 2.54мм:PINHD-1X1
- added R27, R28, R31: 330, rcl:R-EU_M0805
- added R29, R30: 620, rcl:R-EU_M0805
- added R33: 1k5, rcl:R-EU_M0805
- added R34: 1k, rcl:R-EU_M0805
- added R35: 3k3, rcl:R-EU_M0805
- added VD1, VD3, VD4, VD5: КД521, diode:DIODE-D-7.5
- added VT2: КТ315, m_transistor:BJT_NPN_TO-92_ECB
- C12: value (none) -> 8..30
Connections:
- new net N$100: L2A.1, VT2.C
- new net N$101: DD1D.O, R33.2
- new net N$102: R35.2, VD4.C, VD6.C
- new net N$91: C6.2, C7.1, R21.2
- new net N$92: C13.2, DD4.3.!OUT, L1.2, R27.2
- new net N$93: C12.E, L1.1
- new net N$94: C17.2, VD5.C, VT2.B
- new net N$95: C14.1, DD4.3.OUT, R28.2, R29.2
- new net N$96: C14.2, R30.2, R31.2, VT2.E
- new net N$97: R29.1, R30.1
- new net N$98: R28.1, R31.1
- net A: now also C10.1, C11.1, C13.1, C16.+, C17.1, C18.2, C8.1, DD4P.GND, L2B.1, VD5.A
- net GND: now also C16.-, C18.1, C7.2, DD4P.VCC, R34.1, R35.1
- net N$54: now also C6.1, DD1D.I, R33.1, R34.2, VD4.A
- net N$80: now also C8.2, DD4.1.!OUT, DD4.2.!IN, R15.2, VD1.C
- net N$85: now also C10.2, DD4.2.IN, DD4.3.!IN
- net N$86: now also C11.2, C12.A, DD4.3.IN, R27.1; no longer DD4.1.!OUT, DD4.2.!IN, R15.2
- net N$88: now also C2.2
- net N$89: now also C2.1, VD1.A, VD3.A
Other:
- note added: "RGBS to SECAM RF"
- moved on the sheet: C12, DD1D, DD1E, DD4.1, DD4.2, DD4.3, DD4P, L1, R15, R16, R17, R19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

Commit message: .
Parts:
- removed DD1', DD1'''': 74LS04N, 74xx-eu:74LS04N
- removed R10', R10'', R10''', R10'''', R10'1: 15k, rcl:R-EU_M0805
- removed R11', R11'', R11''', R11'''', R11'1: 7k5, rcl:R-EU_M0805
- removed R12', R12'', R12''', R12'''', R12'1, R4', R4'', R4''', R4'''', R4'1, R7', R7'', R7''', R7'''', R7'1: 5k1, rcl:R-EU_M0805
- removed R13', R13'''', R13'1, R13'2, R13'3: 3k3, rcl:R-EU_M0805
- removed R5', R5'', R5''', R5'''', R5'1: 10k, rcl:R-EU_M0805
- removed R6', R6'', R6''', R6'''', R6'1: 27k, rcl:R-EU_M0805
- removed R8', R8'', R8''', R8'''', R8'1: 33k, rcl:R-EU_M0805
- removed R9', R9'', R9''', R9'''', R9'1: 6k2, rcl:R-EU_M0805
- added R32: 620, rcl:R-EU_M0805
Connections:
- removed net N$1: R4''''.2, R5''''.2, R6''''.2
- removed net N$10: R10'.1, R5'.1, R7'.1
- removed net N$101: DD1D.O, R33.2
- removed net N$11: DD1''''A.O, R10''''.1, R5''''.1, R7''''.1
- removed net N$12: R7''''.2, R8''''.2, R9''''.2
- removed net N$13: DD1''''B.O, R11''''.1, R4''''.1
- removed net N$14: DD1''''B.I, R9''''.1
- removed net N$15: R10''''.2, R11''''.2, R12''''.2, R13''''.2
- removed net N$16: DD1''''C.O, R6''''.1
- removed net N$17: DD1''''C.I, R12''''.1, R8''''.1
- removed net N$18: R4'1.2, R5'1.2, R6'1.2
- removed net N$19: R12'1.1
- removed net N$2: R4'.2, R5'.2, R6'.2
- removed net N$20: R4''.2, R5''.2, R6''.2
- removed net N$21: R7'1.2, R8'1.2, R9'1.2
- removed net N$22: R9'1.1
- removed net N$23: R8'1.1
- removed net N$24: R10'1.2, R11'1.2, R12'1.2, R13'1.2
- removed net N$25: R5'1.1
- removed net N$26: R10'1.1
- removed net N$27: R7'1.1
- removed net N$28: R4'1.1
- removed net N$29: R6'1.1
- removed net N$3: DD1'A.I, R11'.1, R4'.1
- removed net N$30: R11'1.1
- removed net N$31: R7''.2, R8''.2, R9''.2
- removed net N$32: R9''.1
- removed net N$33: R8''.1
- removed net N$34: R10''.2, R11''.2, R12''.2, R13'2.2
- removed net N$35: R5''.1
- removed net N$36: R10''.1
- removed net N$37: R7''.1
- removed net N$38: R4''.1
- removed net N$39: R6''.1
- removed net N$4: R7'.2, R8'.2, R9'.2
- removed net N$40: R11''.1
- removed net N$41: R12''.1
- removed net N$42: R4'''.2, R5'''.2, R6'''.2
- removed net N$43: R7'''.2, R8'''.2, R9'''.2
- removed net N$44: R7'''.1
- removed net N$45: R9'''.1
- removed net N$46: R10'''.2, R11'''.2, R12'''.2, R13'3.2
- removed net N$47: R4'''.1
- removed net N$48: R10'''.1
- removed net N$49: R8'''.1
- removed net N$5: DD1'C.I, R6'.1
- removed net N$50: R5'''.1
- removed net N$51: R6'''.1
- removed net N$52: R11'''.1
- removed net N$53: R12'''.1
- removed net N$6: R10'.2, R11'.2, R12'.2, R13'.2
- removed net N$7: DD1'A.O, R9'.1
- removed net N$8: DD1'C.O, R12'.1, R8'.1
- removed net N$9: DD1''''A.I
- net GND: no longer R13''''.1, R13'.1, R13'1.1, R13'2.1, R13'3.1
- net N$102: now also C15.2
- net N$83: now also C15.1, R32.1, VD3.C
- net N$97: now also R32.2
- net N$98: now also DD1D.O, R33.2
Other:
- note removed: "!95.4.5"
- note removed: "!B"
- note removed: "!G"
- note removed: "!R"
- note removed: "!invert"
- note removed: "92.5.4"
- note removed: "93.10.4"
- moved on the sheet: +5V, B, C1, C10, C11, C12, C13, C14, C15, C16, C17, C18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

Commit message: .
Parts:
- added R36: 620, rcl:R-EU_M0805
- C3, C4: device rcl:C-EUC0805K -> rcl:C-EUC0805
- R20: device rcl:R-EU_M0805 -> rcl:R-EU_0207/12
- renumbered !SJ1 to !J1, !SJ2 to !J2, !SJ3 to !J3, SJ1 to J1, SJ2 to J2, SJ3 to J3
Connections:
- net GND: now also C9.1, R36.2; no longer C9.2
- net N$72: now also C9.2; no longer C9.1
- net N$92: now also R36.1
Other:
- moved on the sheet: C9, DD1E, DD3B, DD3D, R16, R26, R27, VD2

Commit message: .
Parts:
- renumbered R19 to R19*
Connections:
- removed net N$72: C9.2, DD2B.Q, R18.1, R26.1, VD2.A
- new net N$1: DD2B.Q, R18.1, R26.2
- net N$81: now also C9.2, R26.1, VD2.A; no longer R26.2
Other:
- moved on the sheet: DD3B, R15, R26, VD1

Commit message: .
Parts:
- DD4: value К500ЛП216 -> К500ЛП216R; device 500:К500ЛП216 -> 500:К500ЛП216R
- R15: device rcl:R-EU_M0805 -> rcl:R-EU_0207/12
Connections:
- new net N$2: R32.1, VD3.C
- net N$83: no longer R32.1, VD3.C
Other:
- moved on the sheet: R32, VD3

Commit message: .
Parts:
- added L2: (no value), rcl:L-US0204/5
Other:
- moved on the sheet: +5V, R37
Changed lines of the file:
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@@
 <grid distance="0.1" unitdist="inch" unit="mil" style="lines" multiple="1" display="yes" altdistance="0.01" altunitdist="inch" altunit="inch"/>
 <layers>
-<layer number="1" name="Top" color="4" fill="1" visible="yes" active="no"/>
-<layer number="2" name="Route2" color="1" fill="3" visible="yes" active="no"/>
-<layer number="3" name="Route3" color="4" fill="3" visible="yes" active="no"/>
-<layer number="4" name="Route4" color="1" fill="4" visible="yes" active="no"/>
-<layer number="5" name="Route5" color="4" fill="4" visible="yes" active="no"/>
-<layer number="6" name="Route6" color="1" fill="8" visible="yes" active="no"/>
-<layer number="7" name="Route7" color="4" fill="8" visible="yes" active="no"/>
-<layer number="8" name="Route8" color="1" fill="2" visible="yes" active="no"/>
-<layer number="9" name="Route9" color="4" fill="2" visible="yes" active="no"/>
-<layer number="10" name="Route10" color="1" fill="7" visible="yes" active="no"/>
-<layer number="11" name="Route11" color="4" fill="7" visible="yes" active="no"/>
-<layer number="12" name="Route12" color="1" fill="5" visible="yes" active="no"/>
-<layer number="13" name="Route13" color="4" fill="5" visible="yes" active="no"/>
-<layer number="14" name="Route14" color="1" fill="6" visible="yes" active="no"/>
-<layer number="15" name="Route15" color="4" fill="6" visible="yes" active="no"/>
-<layer number="16" name="Bottom" color="1" fill="1" visible="yes" active="no"/>
-<layer number="17" name="Pads" color="2" fill="1" visible="yes" active="no"/>
-<layer number="18" name="Vias" color="2" fill="1" visible="yes" active="no"/>
-<layer number="19" name="Unrouted" color="6" fill="1" visible="yes" active="no"/>
-<layer number="20" name="Dimension" color="15" fill="1" visible="yes" active="no"/>
-<layer number="21" name="tPlace" color="7" fill="1" visible="yes" active="no"/>
-<layer number="22" name="bPlace" color="7" fill="1" visible="yes" active="no"/>
-<layer number="23" name="tOrigins" color="15" fill="1" visible="yes" active="no"/>
-<layer number="24" name="bOrigins" color="15" fill="1" visible="yes" active="no"/>
-<layer number="25" name="tNames" color="7" fill="1" visible="yes" active="no"/>
-<layer number="26" name="bNames" color="7" fill="1" visible="yes" active="no"/>
-<layer number="27" name="tValues" color="7" fill="1" visible="yes" active="no"/>
-<layer number="28" name="bValues" color="7" fill="1" visible="yes" active="no"/>
+<layer number="1" name="Top" color="4" fill="1" visible="no" active="no"/>
+<layer number="2" name="Route2" color="1" fill="3" visible="no" active="no"/>
+<layer number="3" name="Route3" color="4" fill="3" visible="no" active="no"/>
+<layer number="4" name="Route4" color="1" fill="4" visible="no" active="no"/>
+<layer number="5" name="Route5" color="4" fill="4" visible="no" active="no"/>
+<layer number="6" name="Route6" color="1" fill="8" visible="no" active="no"/>
+<layer number="7" name="Route7" color="4" fill="8" visible="no" active="no"/>
+<layer number="8" name="Route8" color="1" fill="2" visible="no" active="no"/>
+<layer number="9" name="Route9" color="4" fill="2" visible="no" active="no"/>
+<layer number="10" name="Route10" color="1" fill="7" visible="no" active="no"/>
+<layer number="11" name="Route11" color="4" fill="7" visible="no" active="no"/>
+<layer number="12" name="Route12" color="1" fill="5" visible="no" active="no"/>
+<layer number="13" name="Route13" color="4" fill="5" visible="no" active="no"/>
+<layer number="14" name="Route14" color="1" fill="6" visible="no" active="no"/>
+<layer number="15" name="Route15" color="4" fill="6" visible="no" active="no"/>
+<layer number="16" name="Bottom" color="1" fill="1" visible="no" active="no"/>
+<layer number="17" name="Pads" color="2" fill="1" visible="no" active="no"/>
+<layer number="18" name="Vias" color="2" fill="1" visible="no" active="no"/>
+<layer number="19" name="Unrouted" color="6" fill="1" visible="no" active="no"/>
+<layer number="20" name="Dimension" color="15" fill="1" visible="no" active="no"/>
+<layer number="21" name="tPlace" color="7" fill="1" visible="no" active="no"/>
+<layer number="22" name="bPlace" color="7" fill="1" visible="no" active="no"/>
+<layer number="23" name="tOrigins" color="15" fill="1" visible="no" active="no"/>
+<layer number="24" name="bOrigins" color="15" fill="1" visible="no" active="no"/>
+<layer number="25" name="tNames" color="7" fill="1" visible="no" active="no"/>
+<layer number="26" name="bNames" color="7" fill="1" visible="no" active="no"/>
+<layer number="27" name="tValues" color="7" fill="1" visible="no" active="no"/>
+<layer number="28" name="bValues" color="7" fill="1" visible="no" active="no"/>
 <layer number="29" name="tStop" color="7" fill="3" visible="no" active="no"/>
 <layer number="30" name="bStop" color="7" fill="6" visible="no" active="no"/>
@@
 <layer number="35" name="tGlue" color="7" fill="4" visible="no" active="no"/>
 <layer number="36" name="bGlue" color="7" fill="5" visible="no" active="no"/>
-<layer number="37" name="tTest" color="7" fill="1" visible="yes" active="no"/>
-<layer number="38" name="bTest" color="7" fill="1" visible="yes" active="no"/>
+<layer number="37" name="tTest" color="7" fill="1" visible="no" active="no"/>
+<layer number="38" name="bTest" color="7" fill="1" visible="no" active="no"/>
 <layer number="39" name="tKeepout" color="4" fill="11" visible="no" active="no"/>
 <layer number="40" name="bKeepout" color="1" fill="11" visible="no" active="no"/>
@@
 <layer number="44" name="Drills" color="7" fill="1" visible="no" active="no"/>
 <layer number="45" name="Holes" color="7" fill="1" visible="no" active="no"/>
-<layer number="46" name="Milling" color="3" fill="1" visible="yes" active="no"/>
-<layer number="47" name="Measures" color="7" fill="1" visible="yes" active="no"/>
-<layer number="48" name="Document" color="7" fill="1" visible="yes" active="no"/>
-<layer number="49" name="Reference" color="7" fill="1" visible="yes" active="no"/>
-<layer number="50" name="dxf" color="7" fill="1" visible="yes" active="no"/>
-<layer number="51" name="tDocu" color="7" fill="1" visible="yes" active="no"/>
-<layer number="52" name="bDocu" color="7" fill="1" visible="yes" active="no"/>
-<layer number="53" name="tGND_GNDA" color="7" fill="9" visible="yes" active="no"/>
-<layer number="54" name="bGND_GNDA" color="1" fill="9" visible="yes" active="no"/>
-<layer number="56" name="wert" color="7" fill="1" visible="yes" active="no"/>
-<layer number="57" name="tCAD" color="7" fill="1" visible="yes" active="no"/>
+<layer number="46" name="Milling" color="3" fill="1" visible="no" active="no"/>
+<layer number="47" name="Measures" color="7" fill="1" visible="no" active="no"/>
+<layer number="48" name="Document" color="7" fill="1" visible="no" active="no"/>
+<layer number="49" name="Reference" color="7" fill="1" visible="no" active="no"/>
+<layer number="50" name="dxf" color="7" fill="1" visible="no" active="no"/>
+<layer number="51" name="tDocu" color="7" fill="1" visible="no" active="no"/>
+<layer number="52" name="bDocu" color="7" fill="1" visible="no" active="no"/>
+<layer number="53" name="tGND_GNDA" color="7" fill="9" visible="no" active="no"/>
+<layer number="54" name="bGND_GNDA" color="1" fill="9" visible="no" active="no"/>
+<layer number="56" name="wert" color="7" fill="1" visible="no" active="no"/>
+<layer number="57" name="tCAD" color="7" fill="1" visible="no" active="no"/>
 <layer number="90" name="Modules" color="5" fill="1" visible="yes" active="yes"/>
 <layer number="91" name="Nets" color="2" fill="1" visible="yes" active="yes"/>
@@
 <part name="R36" library="rcl" deviceset="R-EU_" device="M0805" value="620"/>
 <part name="GND1" library="supply1v" deviceset="GND" device=""/>
+<part name="L2" library="rcl" deviceset="L-US" device="0204/5"/>
 </parts>
 <sheets>
@@
 <instance part="DD3" gate="P" x="45.72" y="86.36"/>
 <instance part="DD1" gate="P" x="30.48" y="86.36"/>
-<instance part="R37" gate="G$1" x="38.1" y="104.14" rot="R90"/>
+<instance part="R37" gate="G$1" x="17.78" y="109.22" rot="R90"/>
 <instance part="GND8" gate="1" x="38.1" y="71.12"/>
-<instance part="+5V" gate="G$1" x="38.1" y="119.38" smashed="yes" rot="R90">
-<attribute name="NAME" x="39.37" y="123.825" size="1.778" layer="95" rot="R180"/>
-<attribute name="VALUE" x="43.18" y="113.03" size="1.778" layer="96" rot="R90"/>
+<instance part="+5V" gate="G$1" x="17.78" y="124.46" smashed="yes" rot="R90">
+<attribute name="NAME" x="19.05" y="128.905" size="1.778" layer="95" rot="R180"/>
+<attribute name="VALUE" x="22.86" y="118.11" size="1.778" layer="96" rot="R90"/>
 </instance>
 <instance part="VT1" gate="G$1" x="22.86" y="66.04" smashed="yes">
@@
 <instance part="R36" gate="G$1" x="223.52" y="152.4"/>
 <instance part="GND1" gate="1" x="233.68" y="152.4" rot="R90"/>
+<instance part="L2" gate="G$1" x="45.72" y="111.76" rot="R90"/>
 </instances>
 <busses>
@@
 <wire x1="45.72" y1="96.52" x2="45.72" y2="93.98" width="0.1524" layer="91"/>
 <pinref part="R37" gate="G$1" pin="1"/>
-<wire x1="38.1" y1="99.06" x2="38.1" y2="96.52" width="0.1524" layer="91"/>
 <junction x="38.1" y="96.52"/>
 <junction x="30.48" y="96.52"/>
@@
 <wire x1="53.34" y1="96.52" x2="45.72" y2="96.52" width="0.1524" layer="91"/>
 <junction x="45.72" y="96.52"/>
+<wire x1="17.78" y1="104.14" x2="17.78" y2="96.52" width="0.1524" layer="91"/>
+<junction x="17.78" y="96.52"/>
 </segment>
 <segment>
@@
 <pinref part="+5V" gate="G$1" pin="1"/>
 <pinref part="R37" gate="G$1" pin="2"/>
-<wire x1="38.1" y1="116.84" x2="38.1" y2="109.22" width="0.1524" layer="91"/>
-</segment>
-</net>
+<wire x1="17.78" y1="121.92" x2="17.78" y2="114.3" width="0.1524" layer="91"/>
+</segment>
+</net>

Commit message: ..
Parts:
- added C19: 50m, rcl:CPOL-EUE2.5-6
- added C20: 100n, rcl:C-EUC0805K
- DD4: value К500ЛП216R -> К500ЛП216
- R37: value 8* -> 8(20r)*
Connections:
- new net B: C10.1, C11.1, C13.1, C16.+, C17.1, C18.2, C8.1, DD4P.GND, L2.2, L2B.1, VD5.A
- net A: now also C19.+, C20.1, L2.1, R37.2; no longer C10.1, C11.1, C13.1, C16.+, C17.1, C18.2, C8.1, DD4P.GND, L2B.1, R37.1, VD5.A
- net GND: now also C19.-, C20.2, C9.2; no longer C9.1
- net N$102: now also VD4.A; no longer VD4.C
- net N$54: now also VD4.C; no longer VD4.A
- net N$76: now also R37.1; no longer R37.2
- net N$81: now also C9.1; no longer C9.2
Other:
- note added: "(SMD) 100ЛП114 100ЛП116 100ЛП216"
- note added: "(SMD) 564КТ3"
- note added: "(SMD) 564ТМ2 (R18 910k)"
- note added: "C12 10pf"
- note added: "DD2 К561КТ3 (CD4066) К176КТ1"
- note added: "DD3 К561ТМ2 (CD4013)"
- note added: "DD4 К500ЛП216 (MC10216) К500ЛП114 К500ЛП116"
- note added: "T1 30ВЧ"
- moved on the sheet: +5V, C15, C3, C4, C5, C9, DD1D, DD1F, DD2B, L2, R14, R18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
